Commit message: v3

File: description/macros.xacro (robot description, xacro)
@@ -16,5 +16,5 @@
                 <origin xyz="${x2} ${y2} ${z2}" rpy="${roll2} ${pitch2} ${yaw2}"/>
                 <geometry>
-                    <mesh filename="package://xe_tang/meshes/${link_name}.stl"/>
+                    <mesh filename="package://bonbanhomni/meshes/${link_name}.stl"/>
                 </geometry>
                 <material name="${link_name}_material">
@@ -25,5 +25,5 @@
                 <origin xyz="${x2} ${y2} ${z2}" rpy="${roll2} ${pitch2} ${yaw2}"/>
                 <geometry>
-                    <mesh filename="package://xe_tang/meshes/${link_name}.stl"/>
+                    <mesh filename="package://bonbanhomni/meshes/${link_name}.stl"/>
                 </geometry>
             </collision>
